Commit message: Fixed trailer drift in gazebo fortress

File: scout_nav2_gz/urdf/scout_v2/scout_v2_trailer.xacro (robot description, xacro)
@@ -18,5 +18,5 @@
     <xacro:property name="wheel_mass" value="0.6"/>
     <xacro:property name="trailer_wheel_length" value="0.045" />
-    <xacro:property name="trailer_wheel_radius" value="0.06" />
+    <xacro:property name="trailer_wheel_radius" value="0.065" />
     <xacro:property name="trailer_wheel_mass" value="0.6"/>
     <xacro:property name="connector_length" value="0.15"/>
@@ -244,7 +244,8 @@
   </joint>
   <!-- Trailer Wheels -->
+  <!--
   <xacro:trailer_wheel prefix="trailer_wheel_lf" x_reflect="1" y_reflect="1" wheel_offset="${trailer_length / 4}"/>
+  <xacro:trailer_wheel prefix="trailer_wheel_rf" x_reflect="1" y_reflect="-1" wheel_offset="${trailer_length / 4}"/>-->
   <xacro:trailer_wheel prefix="trailer_wheel_lr" x_reflect="-1" y_reflect="1" wheel_offset="${trailer_length / 4}"/>
-  <xacro:trailer_wheel prefix="trailer_wheel_rf" x_reflect="1" y_reflect="-1" wheel_offset="${trailer_length / 4}"/>
   <xacro:trailer_wheel prefix="trailer_wheel_rr" x_reflect="-1" y_reflect="-1" wheel_offset="${trailer_length / 4}"/>
     <!-- IMU -->

Commit message: trailer is published but not rotating

File: scout_nav2_gz/urdf/scout_v2/scout_v2_trailer.xacro (robot description, xacro)
@@ -214,5 +214,6 @@
     <origin xyz="${(-base_x_size/2)} 0 -0.065 " rpy="0 0 0"/>
     <axis xyz="0 0 1"/>
-    <limit effort="100" velocity="2.0" lower="${-pi/4}" upper="${pi/4}"/>
+    <limit effort="0.0" velocity="10.0" lower="${-pi/4}" upper="${pi/4}"/>
+    <dynamics damping="0.1"/>
   </joint>
   <!-- Trailer Link -->

Commit message: testing remote pushes

File: scout_nav2_gz/urdf/scout_v2/scout_v2_trailer.xacro (robot description, xacro)
@@ -212,9 +212,26 @@
     <parent link="base_link"/>
     <child link="trailer_connector_link"/>
-    <origin xyz="${(-base_x_size/2)} 0 -0.065 " rpy="0 0 0"/>
+    <origin xyz="${(-base_x_size/2)} 0 -0.065" rpy="0 0 0"/>
     <axis xyz="0 0 1"/>
-    <limit effort="0.0" velocity="10.0" lower="${-pi/4}" upper="${pi/4}"/>
-    <dynamics damping="0.1"/>
-  </joint>
+    <limit effort="0.0" velocity="10.0" lower="-1.57" upper="1.57"/>
+    <dynamics damping="0.05" friction="0.1"/>
+  </joint>
+  <gazebo reference="trailer_connector_joint">
+    <dynamics damping="0.05" friction="0.1"/>
+    <physics>
+      <ode>
+        <limit>
+          <cfm>0.1</cfm>
+          <erp>0.9</erp>
+        </limit>
+      </ode>
+    </physics>
+  </gazebo>
+  <!-- <joint name="trailer_connector_joint" type="fixed">
+    <parent link="base_link"/>
+    <child link="trailer_connector_link"/>
+    <origin xyz="${(-base_x_size/2)} 0 -0.065" rpy="0 0 0"/>
+    <axis xyz="0 0 1"/>
+  </joint> -->
   <!-- Trailer Link -->
   <link name="trailer_link">

Commit message: tried changing everything to static

File: scout_nav2_gz/urdf/scout_v2/scout_v2_trailer.xacro (robot description, xacro)
@@ -241,5 +241,4 @@
     <origin xyz="${-(connector_length)} 0 0" rpy="0 0 0"/>
     <axis xyz="0 0 1"/>
-    <limit effort="100" lower="-3.14159" upper="3.14159" velocity="1"/>
   </joint>
   <!-- Trailer Wheels -->
