Commit message: started transfering to gazebo classic

File: scout_description/urdf/scout_v2/scout_v2_trailer.xacro (robot description, xacro)
@@ -18,5 +18,5 @@
     <xacro:property name="wheel_mass" value="0.6"/>
     <xacro:property name="trailer_wheel_length" value="0.045" />
-    <xacro:property name="trailer_wheel_radius" value="0.06" />
+    <xacro:property name="trailer_wheel_radius" value="0.065" />
     <xacro:property name="trailer_wheel_mass" value="0.6"/>
     <xacro:property name="connector_length" value="0.15"/>
@@ -109,4 +109,52 @@
         <origin xyz="${-wheelbase/2} ${-track/2} ${wheel_vertical_offset}" rpy="3.14 0 0" />
     </xacro:scout_wheel_type2>
+    <!-- Camera stand box -->
+  <link name="camera_stand_link">
+      <visual>
+          <origin xyz="0 0 0" rpy="0 0 0"/>
+          <geometry>
+              <box size="0.15 0.15 0.01"/> <!-- Adjust size as needed -->
+          </geometry>
+          <material name="Gray">
+              <color rgba="0.5 0.5 0.5 1.0"/>
+          </material>
+      </visual>
+      <collision>
+          <origin xyz="0 0 0" rpy="0 0 0"/>
+          <geometry>
+              <box size="0.15 0.15 0.01"/> <!-- Same size for collision -->
+          </geometry>
+      </collision>
+      <xacro:box_inertia m="0.1" w="0.1" d="0.1" h="0.1"/>
+  </link>
+  <joint name="camera_stand_joint" type="fixed">
+      <parent link="base_link"/>
+      <child link="camera_stand_link"/>
+      <origin xyz="0.24 0 ${(base_z_size/2) + 0.0127}" rpy="0 0 0"/>
+  </joint>
+  <!-- Lidar stand box -->
+  <link name="lidar_stand_link">
+      <visual>
+          <origin xyz="0 0 0" rpy="0 0 0"/>
+          <geometry>
+              <box size="0.1 0.15 0.04"/> <!-- Adjust size as needed -->
+          </geometry>
+          <material name="Gray">
+              <color rgba="0.5 0.5 0.5 1.0"/>
+          </material>
+      </visual>
+      <collision>
+          <origin xyz="0 0 0" rpy="0 0 0"/>
+          <geometry>
+              <box size="0.1 0.15 0.04"/> <!-- Same size for collision -->
+          </geometry>
+      </collision>
+      <xacro:box_inertia m="0.1" w="0.1" d="0.1" h="0.1"/>
+  </link>
+  <joint name="lidar_stand_joint" type="fixed">
+      <parent link="camera_stand_link"/>
+      <child link="lidar_stand_link"/>
+      <origin xyz="-0.01 0 0.025" rpy="0 0 0"/>
+  </joint>
     <!--                TRAILER             -->
     <!-- Trailer wheel macro -->
@@ -196,7 +244,8 @@
   </joint>
   <!-- Trailer Wheels -->
+  <!--
   <xacro:trailer_wheel prefix="trailer_wheel_lf" x_reflect="1" y_reflect="1" wheel_offset="${trailer_length / 4}"/>
+  <xacro:trailer_wheel prefix="trailer_wheel_rf" x_reflect="1" y_reflect="-1" wheel_offset="${trailer_length / 4}"/>-->
   <xacro:trailer_wheel prefix="trailer_wheel_lr" x_reflect="-1" y_reflect="1" wheel_offset="${trailer_length / 4}"/>
-  <xacro:trailer_wheel prefix="trailer_wheel_rf" x_reflect="1" y_reflect="-1" wheel_offset="${trailer_length / 4}"/>
   <xacro:trailer_wheel prefix="trailer_wheel_rr" x_reflect="-1" y_reflect="-1" wheel_offset="${trailer_length / 4}"/>
     <!-- IMU -->
@@ -320,50 +369,29 @@
         </plugin>
     </gazebo>
-<!--     <gazebo>
-        <plugin name="skid_steer_drive_controller" filename="libgazebo_ros_skid_steer_drive.so">
-            <updateRate>100.0</updateRate>
-            <robotNamespace></robotNamespace>
-            <leftFrontJoint>front_left_wheel</leftFrontJoint>
-            <rightFrontJoint>front_right_wheel</rightFrontJoint>
-            <leftRearJoint>rear_left_wheel</leftRearJoint>
-            <rightRearJoint>rear_right_wheel</rightRearJoint>
-            <wheelSeparation>4</wheelSeparation>
-            <wheelDiameter>0.32918</wheelDiameter>
-            <robotBaseFrame>base_link</robotBaseFrame>
-            <torque>1000</torque>
-            <commandTopic>cmd_vel</commandTopic>
-            <broadcastTF>true</broadcastTF>
-            <odometryTopic>odom</odometryTopic>
-            <odometryFrame>odom</odometryFrame>
-            <covariance_x>0.000100</covariance_x>
-            <covariance_y>0.000100</covariance_y>
-            <covariance_yaw>0.010000</covariance_yaw>
-        </plugin>
-    </gazebo> -->
     <!-- LIDAR -->
     <link name="lidar_link">
-        <inertial>
-        <origin xyz="0 0 0" rpy="0 0 0"/>
-        <mass value="0.125"/>
-        <inertia ixx="0.001"  ixy="0"  ixz="0" iyy="0.001" iyz="0" izz="0.001" />
-        </inertial>
-        <collision>
-        <origin xyz="0 0 0" rpy="0 0 0"/>
-        <geometry>
-            <cylinder radius="0.0254" length="0.0275"/>
-        </geometry>
-        </collision>
-        <visual>
-        <origin xyz="0 0 0" rpy="0 0 0"/>
-        <geometry>
-            <cylinder radius="0.0254" length="0.0275"/>
-        </geometry>
-        </visual>
-    </link>
-    <joint name="lidar_joint" type="fixed">
+    <inertial>
+      <origin xyz="0 0 0" rpy="0 0 0"/>
+      <mass value="0.125"/>
+      <inertia ixx="0.001"  ixy="0"  ixz="0" iyy="0.001" iyz="0" izz="0.001" />
+    </inertial>
+    <collision>
+      <origin xyz="0 0 0" rpy="0 0 0"/>
+      <geometry>
+        <cylinder radius="0.06" length="0.086"/>
+      </geometry>
+    </collision>
+    <visual>
+      <origin xyz="0 0 0" rpy="0 0 0"/>
+      <geometry>
+        <cylinder radius="0.06" length="0.086"/>
+      </geometry>
+    </visual>
+  </link>
+  <joint name="lidar_joint" type="fixed">
         <parent link="base_link"/>
         <child link="lidar_link"/>
-        <origin xyz="0.4 0 ${(base_z_size/2) + 0.02 + 0.0275}" rpy="0 0 0"/>
-    </joint>
+        <origin xyz="0.25 0 ${(base_z_size/2) + 0.0127 + 0.025 + 0.02 + (0.086/2)}" rpy="0 0 0"/>
+  </joint>
     <gazebo reference="lidar_link">
         <sensor name="lidar" type="ray">
@@ -382,5 +410,5 @@
             <range>
             <min>0.150000</min>
-            <max>12</max>
+            <max>20</max>
             <resolution>0.015000</resolution>
             </range>
@@ -423,7 +451,7 @@
     </link>
     <joint name="camera_joint" type="fixed">
-        <parent link="base_link"/>
+        <parent link="camera_stand_link"/>
         <child link="camera_link"/>
-        <origin xyz="0.4 0 ${(base_z_size/2) + 0.02}" rpy="0 0 0"/>
+        <origin xyz="0.06 0 0.02" rpy="0 0 0"/>
     </joint>
     <link name="camera_depth_frame"/>

File: scout_nav2_gz/urdf/scout_v2/scout_v2_trailer.xacro (robot description, xacro)
@@ -214,5 +214,5 @@
     <origin xyz="${(-base_x_size/2)} 0 -0.065 " rpy="0 0 0"/>
     <axis xyz="0 0 1"/>
-    <limit effort="100" velocity="2.0" lower="${-pi/4}" upper="${pi/4}"/>
+    <limit effort="1000" velocity="1000.0" lower="${-pi/4}" upper="${pi/4}"/>
   </joint>
   <!-- Trailer Link -->

Commit message: comoletly transfered to classic

File: scout_description/urdf/scout_v2/scout_v2_trailer.xacro (robot description, xacro)
@@ -157,37 +157,37 @@
       <origin xyz="-0.01 0 0.025" rpy="0 0 0"/>
   </joint>
-    <!--                TRAILER             -->
-    <!-- Trailer wheel macro -->
-    <xacro:macro name="trailer_wheel" params="prefix x_reflect y_reflect wheel_offset">
-        <link name="${prefix}_link">
-        <visual>
-            <geometry>
-            <cylinder radius="${trailer_wheel_radius}" length="${trailer_wheel_length}"/>
-            </geometry>
-            <origin xyz="0 0 0" rpy="${pi/2} ${pi/2} 0"/>
-            <material name="Gray">
-            <color rgba="0.5 0.5 0.5 1.0"/>
-            </material>
-        </visual>
-        <collision>
-            <geometry>
-            <cylinder radius="${trailer_wheel_radius}" length="${trailer_wheel_length}"/>
-            </geometry>
-            <origin xyz="0 0 0" rpy="${pi/2} ${pi/2} 0"/>
-        </collision>
-        <xacro:cylinder_inertia m="${trailer_wheel_mass}" r="${trailer_wheel_radius}" h="${trailer_wheel_length}"/>
-        </link>
-        <gazebo reference="${prefix}_link">
-            <mu1>0.1</mu1>
-            <mu2>0.1</mu2>
-        </gazebo>
-        <joint name="${prefix}_joint" type="continuous">
-        <parent link="trailer_link"/>
-        <child link="${prefix}_link"/>
-        <origin xyz="${(x_reflect * wheel_offset) - (trailer_length/2)} ${y_reflect * (trailer_width / 2 + trailer_wheel_length / 2)} ${-trailer_height / 2}" rpy="0 0 0"/>
-        <axis xyz="0 1 0"/>
-        </joint>
-    </xacro:macro>
-    <!-- Trailer Connector Link -->
+   <!--                TRAILER             -->
+  <!-- Trailer wheel macro -->
+  <xacro:macro name="trailer_wheel" params="prefix x_reflect y_reflect wheel_offset">
+    <link name="${prefix}_link">
+      <visual>
+        <geometry>
+          <cylinder radius="${trailer_wheel_radius}" length="${trailer_wheel_length}"/>
+        </geometry>
+        <origin xyz="0 0 0" rpy="${pi/2} ${pi/2} 0"/>
+        <material name="Gray">
+          <color rgba="0.5 0.5 0.5 1.0"/>
+        </material>
+      </visual>
+      <collision>
+        <geometry>
+          <cylinder radius="${trailer_wheel_radius}" length="${trailer_wheel_length}"/>
+        </geometry>
+        <origin xyz="0 0 0" rpy="${pi/2} ${pi/2} 0"/>
+      </collision>
+      <xacro:cylinder_inertia m="${trailer_wheel_mass}" r="${trailer_wheel_radius}" h="${trailer_wheel_length}"/>
+    </link>
+    <gazebo reference="${prefix}_link">
+      <mu1>0.1</mu1>
+      <mu2>0.1</mu2>
+    </gazebo>
+    <joint name="${prefix}_joint" type="continuous">
+      <parent link="trailer_link"/>
+      <child link="${prefix}_link"/>
+      <origin xyz="${(x_reflect * wheel_offset) - (trailer_length/2)} ${y_reflect * (trailer_width / 2 + trailer_wheel_length / 2)} ${-trailer_height / 2}" rpy="0 0 0"/>
+      <axis xyz="0 1 0"/>
+    </joint>
+  </xacro:macro>
+  <!-- Trailer Connector Link -->
     <link name="trailer_connector_link">
     <visual>
@@ -214,5 +214,5 @@
     <origin xyz="${(-base_x_size/2)} 0 -0.065 " rpy="0 0 0"/>
     <axis xyz="0 0 1"/>
-    <limit effort="100" velocity="2.0" lower="${-pi/4}" upper="${pi/4}"/>
+    <limit effort="1000" velocity="1000.0" lower="${-pi/4}" upper="${pi/4}"/>
   </joint>
   <!-- Trailer Link -->
@@ -241,5 +241,4 @@
     <origin xyz="${-(connector_length)} 0 0" rpy="0 0 0"/>
     <axis xyz="0 0 1"/>
-    <limit effort="100" lower="-3.14159" upper="3.14159" velocity="1"/>
   </joint>
   <!-- Trailer Wheels -->
@@ -272,6 +271,5 @@
         <plugin filename="libgazebo_ros_imu_sensor.so" name="imu_plugin">
             <ros>
-            <!-- <namespace>/demo</namespace> -->
-            <remapping>~/out:=imu</remapping>
+                <remapping>~/out:=imu</remapping>
             </ros>
             <initial_orientation_as_reference>false</initial_orientation_as_reference>
@@ -357,8 +355,8 @@
         <max_wheel_torque>1000</max_wheel_torque>
         <max_wheel_acceleration>1.0</max_wheel_acceleration>
-        <updateRate>100</updateRate>
+        <!-- <updateRate>100</updateRate>
         <covariance_x>0.000100</covariance_x>
         <covariance_y>0.000100</covariance_y>
-        <covariance_yaw>0.010000</covariance_yaw>
+        <covariance_yaw>0.010000</covariance_yaw> -->
         <!-- output -->
         <publish_odom>true</publish_odom>
@@ -397,29 +395,29 @@
         <sensor name="lidar" type="ray">
         <always_on>true</always_on>
-        <visualize>false</visualize>
+        <visualize>true</visualize>
         <update_rate>5</update_rate>
         <ray>
             <scan>
-            <horizontal>
-                <samples>360</samples>
-                <resolution>1.000000</resolution>
-                <min_angle>0.000000</min_angle>
-                <max_angle>6.280000</max_angle>
-            </horizontal>
+                <horizontal>
+                    <samples>360</samples>
+                    <resolution>1.000000</resolution>
+                    <min_angle>0.000000</min_angle>
+                    <max_angle>6.280000</max_angle>
+                </horizontal>
             </scan>
             <range>
-            <min>0.150000</min>
-            <max>20</max>
-            <resolution>0.015000</resolution>
+                <min>0.150000</min>
+                <max>30</max>
+                <resolution>0.015000</resolution>
             </range>
             <noise>
-            <type>gaussian</type>
-            <mean>0.0</mean>
-            <stddev>0.01</stddev>
+                <type>gaussian</type>
+                <mean>0.0</mean>
+                <stddev>0.01</stddev>
             </noise>
         </ray>
         <plugin name="scan" filename="libgazebo_ros_ray_sensor.so">
             <ros>
-            <remapping>~/out:=scan</remapping>
+                <remapping>~/out:=scan</remapping>
             </ros>
             <output_type>sensor_msgs/LaserScan</output_type>

Commit message: prot to classic done

File: scout_description/urdf/scout_v2/scout_v2_trailer.xacro (robot description, xacro)
@@ -214,5 +214,5 @@
     <origin xyz="${(-base_x_size/2)} 0 -0.065 " rpy="0 0 0"/>
     <axis xyz="0 0 1"/>
-    <limit effort="1000" velocity="1000.0" lower="${-pi/4}" upper="${pi/4}"/>
+    <limit effort="0.0" velocity="1000.0" lower="${-0.7854}" upper="${0.7853}"/>
   </joint>
   <!-- Trailer Link -->

Commit message: fix: trailer no fricton fix again? 0.07 now wr

File: scout_description/urdf/scout_v2/scout_v2_trailer.xacro (robot description, xacro)
@@ -18,5 +18,6 @@
     <xacro:property name="wheel_mass" value="0.6"/>
     <xacro:property name="trailer_wheel_length" value="0.045" />
-    <xacro:property name="trailer_wheel_radius" value="0.065" />
+    <!-- <xacro:property name="trailer_wheel_radius" value="0.065" /> -->
+    <xacro:property name="trailer_wheel_radius" value="0.07" />
     <xacro:property name="trailer_wheel_mass" value="0.6"/>
     <xacro:property name="connector_length" value="0.15"/>
@@ -214,5 +215,5 @@
     <origin xyz="${(-base_x_size/2)} 0 -0.065 " rpy="0 0 0"/>
     <axis xyz="0 0 1"/>
-    <limit effort="0.0" velocity="1000.0" lower="${-0.7854}" upper="${0.7853}"/>
+    <limit effort="1000.0" velocity="1000.0" lower="${-0.7854}" upper="${0.7853}"/>
   </joint>
   <!-- Trailer Link -->

Commit message: fixed lidar problem with the trailer wheels and spawn angle for new world

File: scout_description/urdf/scout_v2/scout_v2_trailer.xacro (robot description, xacro)
@@ -19,5 +19,5 @@
     <xacro:property name="trailer_wheel_length" value="0.045" />
     <!-- <xacro:property name="trailer_wheel_radius" value="0.065" /> -->
-    <xacro:property name="trailer_wheel_radius" value="0.07" />
+    <xacro:property name="trailer_wheel_radius" value="0.067" />
     <xacro:property name="trailer_wheel_mass" value="0.6"/>
     <xacro:property name="connector_length" value="0.15"/>

Commit message: backup for static transformer

File: scout_description/urdf/scout_v2/scout_v2_trailer.xacro (robot description, xacro)
@@ -215,5 +215,5 @@
     <origin xyz="${(-base_x_size/2)} 0 -0.065 " rpy="0 0 0"/>
     <axis xyz="0 0 1"/>
-    <limit effort="1000.0" velocity="1000.0" lower="${-0.7854}" upper="${0.7853}"/>
+    <limit effort="0.0" velocity="1000.0" lower="${-0.7854}" upper="${0.7854}"/>
   </joint>
   <!-- Trailer Link -->

Commit message: now using gps

File: scout_description/urdf/scout_v2/scout_v2_trailer.xacro (robot description, xacro)
@@ -496,3 +496,39 @@
         </sensor>
     </gazebo>
+    <!-- GPS -->
+    <link name="gps_link">
+        <visual>
+            <geometry>
+                <box size="0.01 0.01 0.01"/>
+            </geometry>
+        </visual>
+        <collision>
+            <geometry>
+                <box size="0.01 0.01 0.01"/>
+            </geometry>
+        </collision>
+        <xacro:box_inertia m="0.1" w="0.1" d="0.1" h="0.1"/>
+    </link>
+    <joint name="gps_joint" type="fixed">
+        <parent link="base_link"/>
+        <child link="gps_link"/>
+        <origin xyz="0.0 0.0 0.0"/>
+    </joint>
+    <gazebo reference="gps_link">
+        <sensor name="gps" type="gps">
+            <plugin filename="libgazebo_ros_gps_sensor.so" name="gps_plugin">
+                <ros>
+                    <remapping>~/out:=gps</remapping>
+                </ros>
+                <gps>
+                    <horizontal_position_noise>0.1</horizontal_position_noise>
+                    <vertical_position_noise>0.1</vertical_position_noise>
+                    <horizontal_velocity_noise>0.1</horizontal_velocity_noise>
+                    <vertical_velocity_noise>0.1</vertical_velocity_noise>
+                </gps>
+            </plugin>
+            <always_on>true</always_on>
+            <update_rate>5.0</update_rate>
+        </sensor>
+    </gazebo>
 </robot>

Commit message: changes before map atleration

File: scout_description/urdf/scout_v2/scout_v2_trailer.xacro (robot description, xacro)
@@ -499,45 +499,40 @@
     <link name="gps_link">
         <visual>
+            <origin xyz="0 0 0" rpy="0 0 0"/>
             <geometry>
-                <box size="0.01 0.01 0.01"/>
+                <box size="0.05 0.05 0.02"/>
             </geometry>
+            <material name="Black">
+                <color rgba="0.1 0.1 0.1 1.0"/>
+            </material>
         </visual>
         <collision>
+            <origin xyz="0 0 0" rpy="0 0 0"/>
             <geometry>
-                <box size="0.01 0.01 0.01"/>
+                <box size="0.05 0.05 0.02"/>
             </geometry>
         </collision>
-        <xacro:box_inertia m="0.1" w="0.1" d="0.1" h="0.1"/>
+        <xacro:box_inertia m="0.1" w="0.05" d="0.05" h="0.02"/>
     </link>
     <joint name="gps_joint" type="fixed">
-        <parent link="base_link"/>
+        <parent link="camera_stand_link"/>
         <child link="gps_link"/>
-        <origin xyz="0.0 0.0 0.0"/>
+        <origin xyz="0 0 0.02" rpy="0 0 0"/>
     </joint>
     <gazebo reference="gps_link">
-        <sensor name="tb3_gps" type="gps">
-            <always_on>true</always_on>
-            <update_rate>1</update_rate>
-            <pose>0 0 0 0 0 0</pose>
+        <sensor type="gps" name="gps">
+            <always_on>1</always_on>
+            <update_rate>1.0</update_rate>
             <gps>
-                <position_sensing>
-                <horizontal>
-                    <noise type="gaussian">
-                    <mean>0.0</mean>
-                    <stddev>0.01</stddev>
-                    </noise>
-                </horizontal>
-                <vertical>
-                    <noise type="gaussian">
-                    <mean>0.0</mean>
-                    <stddev>0.01</stddev>
-                    </noise>
-                </vertical>
-                </position_sensing>
+                <horizontal_position_noise>0.1</horizontal_position_noise>
+                <vertical_position_noise>0.1</vertical_position_noise>
+                <horizontal_velocity_noise>0.1</horizontal_velocity_noise>
+                <vertical_velocity_noise>0.1</vertical_velocity_noise>
             </gps>
-            <plugin name="my_gps_plugin" filename="libgazebo_ros_gps_sensor.so">
+            <plugin name="gps_plugin" filename="libgazebo_ros_gps_sensor.so">
                 <ros>
-                <remapping>~/out:=/gps/fix</remapping>
+                    <remapping>~/out:=/gps/fix</remapping>
                 </ros>
+                <frame_name>gps_link</frame_name>
             </plugin>
         </sensor>
